File: amiga-2000-usb-kb-stamp/amiga-2000-usb-kb-stamp.kicad_pcb (KiCad board)
At the start: 2 copper layers, 55.2 x 53 mm, 14 parts, among them IC1 TXS0104ED, J1 USB3075-30-A, J2 USB_HEADER, J3 CIA, J4 CIA-board, J7 Amiga_Reset, J8 USB1046-GF-0190-L-B-A, J9 USB_BOOT, U1 RP2040_Stamp

Commit message: Add files via upload
Connections:
- IC1 pad 6: Net-(IC1-Pad6) -> (no net)
- IC1 pad 7: Net-(IC1-Pad7) -> GND
- IC1 pad 9: Net-(IC1-Pad9) -> (no net)
- J1 pad 4: Net-(J1-Pad4) -> (no net)
Other:
- board text added: "rev 2"
- board text added: "wiretap 2024"
- board text removed: "rev 0"
- board text removed: "wiretap 2022"
