File: amiga-2000-usb-kb-stamp/amiga-2000-usb-kb-stamp.sch (KiCad schematic (older format))
At the start: 13 parts, among them IC1 TXS0104ED, J1 USB3075-30-A, J2 USB_HEADER, J3 CIA, J4 CIA-board, J7 Amiga_Reset, J8 USB1046-GF-0190-L-B-A, J9 USB_BOOT, U1 RP2040_Stamp

Commit message: Add files via upload
Connections:
- net GND: now also IC1.7 (GND)
Changed lines of the file:
@@
 Sheet 1 1
 Title "A2000 RP2040 Stamp Keyboard Adapter"
-Date "2022-08-19"
-Rev "1"
+Date "2024-01-17"
+Rev "2"
 Comp "wiretap"
 Comment1 ""
@@
 KB_RESET_RAW
 Wire Wire Line
-	3400 5050 3400 5500
+	3400 5050 3400 5250
 Text GLabel 5050 4750 2    50   Input ~ 0
 KB_DATA_RAW
@@
 	1    0    0    -1
 $EndComp
+Wire Wire Line
+	3950 5250 3400 5250
+Connection ~ 3400 5250
+Wire Wire Line
+	3400 5250 3400 5500
 $EndSCHEMATC
